Commit message: completed the gazebo thing with everything properly working including the odom in the rviz2 and the teleop twister thing

File: description/robot.urdf.xacro (robot description, xacro)
@@ -1,4 +1,5 @@
 <?xml version="1.0"?>
 <robot xmlns:xacro="http://www.ros.org/wiki/xacro"  name="robot">
-   <xacro:include filename="robot_core.xacro"/>
+   <xacro:include filename="robot_core.xacro" />
+   <xacro:include filename="gazebo_control.xacro" />
 </robot>

File: description/robot_core.xacro (robot description, xacro)
@@ -38,7 +38,10 @@
      </collision>
      <xacro:inertial_box mass="0.5" x="0.3" y="0.3" z="0.15">
-        <origin xyz="0.15 0 0.75" rpy="0 0 0"/>
+        <origin xyz="0.15 0 0.02" rpy="0 0 0"/><!--z=0.075-->
      </xacro:inertial_box>
 </link>
+<gazebo reference="chassis">
+       <material>Gazebo/White</material>
+</gazebo>
 <!--left wheel link-->
 <joint name="left_wheel_joint" type="continuous">
@@ -64,4 +67,7 @@
     </xacro:inertial_cylinder>
 </link>
+<gazebo reference="left_wheel">
+       <material>Gazebo/Blue</material>
+</gazebo>
 <!--right wheel link-->
 <joint name="right_wheel_joint" type="continuous">
@@ -87,4 +93,7 @@
     </xacro:inertial_cylinder>
 </link>
+<gazebo reference="right_wheel">
+       <material>Gazebo/Blue</material>
+   </gazebo>
 <!--caster wheel link-->
 <joint name="caster_wheel_joint" type="fixed">
@@ -109,3 +118,8 @@
     </xacro:inertial_sphere>
 </link>
+<gazebo reference="caster_wheel">
+       <material>Gazebo/Black</material>
+       <mu1 value="0.001"/>
+       <mu2 value="0.001"/>
+   </gazebo>
 </robot>

Commit message: added lidar to the gazebo

File: description/robot.urdf.xacro (robot description, xacro)
@@ -3,3 +3,4 @@
    <xacro:include filename="robot_core.xacro" />
    <xacro:include filename="gazebo_control.xacro" />
+   <xacro:include filename="lidar.xacro" />
 </robot>

File: description/robot_core.xacro (robot description, xacro)
@@ -13,4 +13,7 @@
 <material name="black">
     <color rgba="0 0 0 1" />
+</material>
+<material name="red">
+    <color rgba="1 0 0 1" />
 </material>
 <!--base link-->
